File: ServoArm/Electronics/arm-controller/arm-controller.kicad_pcb (KiCad board)
At the start: 2 copper layers, 1 part, among them U1 DRV11873

Commit message: Arm WIP.
Parts:
- added C1: 0.1uF, Capacitor_SMD:C_0805_2012Metric, F.Cu at (63.2, 152.4)
- added C2: 0.1uF, Capacitor_SMD:C_0805_2012Metric, F.Cu at (61.0, 156.5)
- added C3: 2.2uF, Capacitor_SMD:C_0805_2012Metric, F.Cu at (61.6, 139.1)
- added C4: 22uF, Capacitor_SMD:C_0805_2012Metric, F.Cu at (66.7, 158.8)
- added H1: MountingHole_Pad, MountingHole:MountingHole_2.7mm, F.Cu at (70.0, 138.0)
- added H2: MountingHole_Pad, MountingHole:MountingHole_2.7mm, F.Cu at (55.0, 159.0)
- added J1: Data, Connector_PinHeader_2.54mm:PinHeader_1x04_P2.54mm_Vertical, F.Cu at (53.3, 143.5)
- added J2: Motor, Connector_PinHeader_2.54mm:PinHeader_1x03_P2.54mm_Vertical, F.Cu at (70.5, 148.6)
- added J3: Power, Connector_PinHeader_2.54mm:PinHeader_1x02_P2.54mm_Vertical, F.Cu at (70.5, 158.8)
- added JP1: Motor RL, Jumper:SolderJumper-3_P1.3mm_Open_Pad1.0x1.5mm, F.Cu at (56.5, 149.3)
- added R1: 8K2, Resistor_SMD:R_0805_2012Metric, F.Cu at (59.7, 139.1)
- moved U1 368.6 mm to (61.3, 146.3), turned to 90 degrees
Connections:
- U1 pad 11: Net-(U1-Pad11) -> +5V
- U1 pad 8: Net-(U1-Pad8) -> GND
Routing:
- net +5V: track 0.00 -> 57.2 mm
- net GND: track 0.00 -> 20.8 mm, vias 0 -> 4
- net Net-(J1-Pad3): track 0.00 -> 13.3 mm
- net Net-(J1-Pad4): track 0.00 -> 12.5 mm
- net Net-(J2-Pad1): track 0.00 -> 9.35 mm
- net Net-(J2-Pad3): track 0.00 -> 8.79 mm
- net Net-(J2-Pad2): track 0.00 -> 7.95 mm
- net Net-(J1-Pad1): track 0.00 -> 7.60 mm
- net Net-(J1-Pad2): track 0.00 -> 6.75 mm
- net Net-(C2-Pad2): track 0.00 -> 6.53 mm
- net Net-(C1-Pad2): track 0.00 -> 4.10 mm
- net Net-(R1-Pad2): track 0.00 -> 3.78 mm
- net Net-(C1-Pad1): track 0.00 -> 3.60 mm
- net Net-(C3-Pad1): track 0.00 -> 3.53 mm
- net Net-(JP1-Pad2): track 0.00 -> 2.61 mm
- added copper zone on F.Cu, net GND
Other:
- board outline added: 22.9 x 27.9 mm
