File: Printed-BLDC-motor/Electronics/L6235-breakout/L6235-breakout.sch (KiCad schematic (older format))
At the start: 31 parts, among them J1 CONTROL, J2 HALL, J3 MOTOR, J4 5V, J5 PWR, U1 L6235PD

Commit message: Gearbox and L6235 updates.
Parts:
- removed C3: 100u, Capacitor_THT:CP_Radial_D6.3mm_P2.50mm, symbol adafruit-new:CPOL-USC
- removed C9: C, Capacitor_SMD:C_0805_2012Metric, symbol Device:C
- removed D3: 1N4148, Diode_SMD:D_0805_2012Metric, symbol Diode:1N4148
- added C3: 100u, Capacitor_THT:C_Radial_D8.0mm_H7.0mm_P3.50mm, symbol Device:CP
- added R13: 1R, Resistor_SMD:R_0805_2012Metric, symbol Device:R
- R5: value 0.33R -> 1R
- R7: value R -> 1R
Connections:
- wire segments 112 -> 116
Changed lines of the file:
@@
-$EndComp
-$Comp
-L Diode:1N4148 D3
-U 1 1 615B9ABB
-P 6075 5050
-F 0 "D3" H 6075 5267 50  0000 C CNN
-F 1 "1N4148" H 6075 5176 50  0000 C CNN
-F 2 "Diode_SMD:D_0805_2012Metric" H 6075 4875 50  0001 C CNN
-F 3 "https://assets.nexperia.com/documents/data-sheet/1N4148_1N4448.pdf" H 6075 5050 50  0001 C CNN
-	1    6075 5050
-	1    0    0    -1
-$EndComp
-$Comp
-L Device:R R7
-U 1 1 615BA7AD
-P 6325 5800
-F 0 "R7" H 6395 5846 50  0000 L CNN
-F 1 "R" H 6395 5755 50  0000 L CNN
-F 2 "Resistor_SMD:R_0805_2012Metric" V 6255 5800 50  0001 C CNN
-F 3 "~" H 6325 5800 50  0001 C CNN
-	1    6325 5800
-	1    0    0    -1
-$EndComp
-$Comp
-L Device:C C9
-U 1 1 615BAFC7
-P 6575 5800
-F 0 "C9" H 6690 5846 50  0000 L CNN
-F 1 "C" H 6690 5755 50  0000 L CNN
-F 2 "Capacitor_SMD:C_0805_2012Metric" H 6613 5650 50  0001 C CNN
-F 3 "~" H 6575 5800 50  0001 C CNN
-	1    6575 5800
-	1    0    0    -1
 $EndComp
 $Comp
@@
 	1    0    0    -1
 $EndComp
-Wire Wire Line
-	3125 3875 3550 3875
 Connection ~ 3125 3875
 Connection ~ 2900 3125
-$Comp
-L adafruit-new:CPOL-USC C3
-U 1 1 615DAAB8
-P 3550 3675
-F 0 "C3" H 3575 3725 45  0000 L CNN
-F 1 "100u" H 3575 3550 45  0000 L CNN
-F 2 "Capacitor_THT:CP_Radial_D6.3mm_P2.50mm" H 3580 3825 20  0001 C CNN
-F 3 "" H 3550 3675 50  0001 C CNN
-	1    3550 3675
-	1    0    0    -1
-$EndComp
 Wire Wire Line
 	3125 3575 3550 3575
 Connection ~ 3125 3575
-Wire Wire Line
-	3550 3875 3900 3875
-Connection ~ 3550 3875
 Wire Wire Line
 	3900 3575 3900 3125
@@
 U 1 1 61613E1F
 P 5275 2925
-F 0 "R5" H 5205 2879 50  0000 R CNN
-F 1 "0.33R" H 5205 2970 50  0000 R CNN
+F 0 "R5" H 5325 3175 50  0000 R CNN
+F 1 "1R" H 5325 3250 50  0000 R CNN
 F 2 "Resistor_SMD:R_0805_2012Metric" V 5205 2925 50  0001 C CNN
 F 3 "~" H 5275 2925 50  0001 C CNN
@@
 	8150 2775 8025 2775
 Wire Wire Line
-	5275 3075 6150 3075
+	5275 3075 5375 3075
 Wire Wire Line
 	5275 2375 5275 2775
@@
 Wire Wire Line
 	5300 1575 6150 1575
+$Comp
+L Device:CP C3
+U 1 1 615C8FC6
+P 3550 3725
+F 0 "C3" H 3668 3771 50  0000 L CNN
+F 1 "100u" H 3668 3680 50  0000 L CNN
+F 2 "Capacitor_THT:C_Radial_D8.0mm_H7.0mm_P3.50mm" H 3588 3575 50  0001 C CNN
+F 3 "~" H 3550 3725 50  0001 C CNN
+	1    3550 3725
+	1    0    0    -1
+$EndComp
+Wire Wire Line
+	3125 3875 3550 3875
+Connection ~ 3550 3875
+Wire Wire Line
+	3550 3875 3900 3875
+$Comp
+L Device:R R7
+U 1 1 615C6A29
+P 5150 2925
+F 0 "R7" H 5300 2900 50  0000 R CNN
+F 1 "1R" H 5300 2975 50  0000 R CNN
+F 2 "Resistor_SMD:R_0805_2012Metric" V 5080 2925 50  0001 C CNN
+F 3 "~" H 5150 2925 50  0001 C CNN
+	1    5150 2925
+	-1   0    0    1
+$EndComp
+$Comp
+L Device:R R13
+U 1 1 615C6F4F
+P 5375 2925
+F 0 "R13" H 5305 2879 50  0000 R CNN
+F 1 "1R" H 5305 2970 50  0000 R CNN
+F 2 "Resistor_SMD:R_0805_2012Metric" V 5305 2925 50  0001 C CNN
+F 3 "~" H 5375 2925 50  0001 C CNN
+	1    5375 2925
+	-1   0    0    1
+$EndComp
+Connection ~ 5375 3075
+Wire Wire Line
+	5375 3075 6150 3075
+Wire Wire Line
+	5275 3075 5150 3075
+Connection ~ 5275 3075
+Wire Wire Line
+	5150 2775 5275 2775
+Connection ~ 5275 2775
+Wire Wire Line
+	5375 2775 5275 2775
 $EndSCHEMATC

Commit message: Latest BLDC driver PCB.
Parts:
- removed J4: 5V, Connector_PinHeader_2.54mm:PinHeader_1x02_P2.54mm_Vertical, symbol Connector:Conn_01x02_Male
- added C9: 100u, Capacitor_THT:C_Radial_D8.0mm_H7.0mm_P3.50mm, symbol Device:CP
- added H1, H2, H3, H4: MountingHole, MountingHole:MountingHole_3.2mm_M3, symbol Mechanical:MountingHole
- added IC1: 7805DT, Package_TO_SOT_SMD:TO-252-2, symbol L6235-breakout-rescue:7805DT-adafruit-new
Connections:
- net +5V: now also C9.1, IC1.2 (VO)
- net GND: now also U1.37 (heatsink), C9.2, IC1.3 (GND)
- net VSS: now also IC1.1 (VI); no longer U1.33 (VSB)
- net at R13.2, R5.2, R7.2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: no longer U1.25 (SENSEB)
Changed lines of the file:
@@
 	7150 1175 7150 1275
-$Comp
-L Connector:Conn_01x02_Male J4
-U 1 1 615B391B
-P 2275 3125
-F 0 "J4" H 2383 3306 50  0000 C CNN
-F 1 "5V" H 2383 3215 50  0000 C CNN
-F 2 "Connector_PinHeader_2.54mm:PinHeader_1x02_P2.54mm_Vertical" H 2275 3125 50  0001 C CNN
-F 3 "~" H 2275 3125 50  0001 C CNN
-	1    2275 3125
-	1    0    0    -1
-$EndComp
 $Comp
 L Connector:Conn_01x02_Male J5
@@
 $EndComp
 $Comp
-L reprapltd-kicad:L6235PD U1
-U 1 1 615B25EC
-P 6650 2125
-F 0 "U1" H 6650 3200 50  0000 C CNN
-F 1 "L6235PD" H 6650 3109 50  0000 C CNN
-F 2 "reprapltd-kicad:SOIC-36_11mmx16mmx3.6mm" H 6650 2125 50  0001 C CNN
-F 3 "" H 6650 2125 50  0001 C CNN
-	1    6650 2125
-	1    0    0    -1
-$EndComp
-$Comp
 L power:GND #PWR0101
 U 1 1 615C4DC4
@@
 	2925 3700 2925 3575
 Wire Wire Line
-	2475 3800 2600 3800
-Wire Wire Line
 	2925 3800 2925 3875
-Wire Wire Line
-	2475 3225 2600 3225
-Wire Wire Line
-	2600 3225 2600 3800
-Connection ~ 2600 3800
-Wire Wire Line
-	2600 3800 2925 3800
-$Comp
-L power:+5V #PWR0104
-U 1 1 615C94C4
-P 2900 3050
-F 0 "#PWR0104" H 2900 2900 50  0001 C CNN
-F 1 "+5V" H 2915 3223 50  0000 C CNN
-F 2 "" H 2900 3050 50  0001 C CNN
-F 3 "" H 2900 3050 50  0001 C CNN
-	1    2900 3050
-	1    0    0    -1
-$EndComp
-Wire Wire Line
-	2475 3125 2900 3125
-Wire Wire Line
-	2900 3125 2900 3050
 Text GLabel 2600 2625 2    50   Input ~ 0
 PHASE3
@@
 Connection ~ 6225 3075
 Wire Wire Line
-	6225 3075 7150 3075
-Wire Wire Line
-	7150 1575 6150 1575
-Connection ~ 6150 1575
+	6225 3075 6800 3075
 $Comp
 L Device:C C2
@@
 Wire Wire Line
 	2925 3875 2925 3900
-$Comp
-L Device:C C4
-U 1 1 615D8F7B
-P 3900 3725
-F 0 "C4" H 4015 3771 50  0000 L CNN
-F 1 "0.1u" H 4015 3680 50  0000 L CNN
-F 2 "Capacitor_SMD:C_0805_2012Metric" H 3938 3575 50  0001 C CNN
-F 3 "~" H 3900 3725 50  0001 C CNN
-	1    3900 3725
-	1    0    0    -1
-$EndComp
 Connection ~ 3125 3875
-Connection ~ 2900 3125
 Wire Wire Line
 	3125 3575 3550 3575
 Connection ~ 3125 3575
-Wire Wire Line
-	3900 3575 3900 3125
-Wire Wire Line
-	2900 3125 3900 3125
 Wire Wire Line
 	2550 1025 2450 1025
@@
 	4775 1550 4775 1500
 Connection ~ 4775 1550
-Wire Wire Line
-	6150 2375 7150 2375
 $Comp
 L Device:R R5
@@
 	-1   0    0    1
 $EndComp
-Connection ~ 6150 2375
 Connection ~ 6150 3075
 Text GLabel 5975 2675 0    50   Input ~ 0
@@
 Wire Wire Line
 	7275 1675 7150 1675
-Wire Wire Line
-	7150 2175 6625 2175
 Wire Wire Line
 	6625 2175 6625 2275
@@
 Text GLabel 7275 2175 2    50   Input ~ 0
 ENABLE
-Wire Wire Line
-	7275 2175 7150 2175
-Connection ~ 7150 2175
 Text GLabel 6050 2175 0    50   Input ~ 0
 HALL1
@@
 	5275 2375 5275 2775
 Wire Wire Line
-	5275 2375 6150 2375
-Wire Wire Line
 	6150 2475 4500 2475
 Wire Wire Line
@@
 	5300 1550 5000 1550
 Connection ~ 5000 1550
-Wire Wire Line
-	5300 1575 6150 1575
 $Comp
 L Device:CP C3
@@
 Wire Wire Line
 	3125 3875 3550 3875
-Connection ~ 3550 3875
-Wire Wire Line
-	3550 3875 3900 3875
 $Comp
 L Device:R R7
@@
 Wire Wire Line
 	5375 2775 5275 2775
+$Comp
+L reprapltd-kicad:L6235PD U1
+U 1 1 616A35F1
+P 6650 2125
+F 0 "U1" H 6650 3200 50  0000 C CNN
+F 1 "L6235PD" H 6650 3109 50  0000 C CNN
+F 2 "reprapltd-kicad:SOIC-36_11mmx16mmx3.6mm" H 6650 2125 50  0001 C CNN
+F 3 "" H 6650 2125 50  0001 C CNN
+	1    6650 2125
+	1    0    0    -1
+$EndComp
+Wire Wire Line
+	5275 2375 6150 2375
+Wire Wire Line
+	6625 2175 7150 2175
+Wire Wire Line
+	5300 1575 6150 1575
+Connection ~ 7150 2175
+Wire Wire Line
+	7150 2175 7275 2175
+Wire Wire Line
+	6650 3125 6800 3125
+Wire Wire Line
+	6800 3125 6800 3075
+Connection ~ 6800 3075
+Wire Wire Line
+	6800 3075 7150 3075
+$Comp
+L L6235-breakout-rescue:7805DT-adafruit-new IC1
+U 1 1 616EDC10
+P 5625 4075
+F 0 "IC1" H 5625 4329 45  0000 C CNN
+F 1 "7805DT" H 5625 4245 45  0000 C CNN
+F 2 "Package_TO_SOT_SMD:TO-252-2" H 5655 4225 20  0001 C CNN
+F 3 "" H 5625 4075 50  0001 C CNN
+	1    5625 4075
+	1    0    0    -1
+$EndComp
+$Comp
+L power:+5V #PWR0104
+U 1 1 616EFB17
+P 6200 4075
+F 0 "#PWR0104" H 6200 3925 50  0001 C CNN
+F 1 "+5V" H 6215 4248 50  0000 C CNN
+F 2 "" H 6200 4075 50  0001 C CNN
+F 3 "" H 6200 4075 50  0001 C CNN
+	1    6200 4075
+	1    0    0    -1
+$EndComp
+$Comp
+L Device:C C4
+U 1 1 616F017A
+P 6325 4225
+F 0 "C4" H 6440 4271 50  0000 L CNN
+F 1 "0.1u" H 6440 4180 50  0000 L CNN
+F 2 "Capacitor_SMD:C_0805_2012Metric" H 6363 4075 50  0001 C CNN
+F 3 "~" H 6325 4225 50  0001 C CNN
+	1    6325 4225
+	1    0    0    -1
+$EndComp
+$Comp
+L power:VSS #PWR0107
+U 1 1 616F094C
+P 5025 4075
+F 0 "#PWR0107" H 5025 3925 50  0001 C CNN
+F 1 "VSS" H 5040 4248 50  0000 C CNN
+F 2 "" H 5025 4075 50  0001 C CNN
+F 3 "" H 5025 4075 50  0001 C CNN
+	1    5025 4075
+	1    0    0    -1
+$EndComp
+$Comp
+L Device:CP C9
+U 1 1 616F1027
+P 6775 4225
+F 0 "C9" H 6893 4271 50  0000 L CNN
+F 1 "100u" H 6893 4180 50  0000 L CNN
+F 2 "Capacitor_THT:C_Radial_D8.0mm_H7.0mm_P3.50mm" H 6813 4075 50  0001 C CNN
+F 3 "~" H 6775 4225 50  0001 C CNN
+	1    6775 4225
+	1    0    0    -1
+$EndComp
+Wire Wire Line
+	2475 3800 2925 3800
+Wire Wire Line
+	5025 4075 5225 4075
+$Comp
+L power:GND #PWR0115
+U 1 1 616F6BB6
+P 5625 4425
+F 0 "#PWR0115" H 5625 4175 50  0001 C CNN
+F 1 "GND" H 5630 4252 50  0000 C CNN
+F 2 "" H 5625 4425 50  0001 C CNN
+F 3 "" H 5625 4425 50  0001 C CNN
+	1    5625 4425
+	1    0    0    -1
+$EndComp
+Wire Wire Line
+	5625 4375 5625 4425
+Wire Wire Line
+	6025 4075 6200 4075
+Wire Wire Line
+	6200 4075 6325 4075
+Connection ~ 6200 4075
+Wire Wire Line
+	6775 4075 6325 4075
+Connection ~ 6325 4075
+Wire Wire Line
+	6775 4375 6325 4375
+Wire Wire Line
+	6325 4375 5625 4375
+Connection ~ 6325 4375
+Connection ~ 5625 4375
+$Comp
+L Mechanical:MountingHole H4
+U 1 1 616F56E4
+P 8350 4850
+F 0 "H4" H 8450 4896 50  0000 L CNN
+F 1 "MountingHole" H 8450 4805 50  0000 L CNN
+F 2 "MountingHole:MountingHole_3.2mm_M3" H 8350 4850 50  0001 C CNN
+F 3 "~" H 8350 4850 50  0001 C CNN
+	1    8350 4850
+	1    0    0    -1
+$EndComp
+$Comp
+L Mechanical:MountingHole H1
+U 1 1 617216E4
+P 7900 5250
+F 0 "H1" H 8000 5296 50  0000 L CNN
+F 1 "MountingHole" H 8000 5205 50  0000 L CNN
+F 2 "MountingHole:MountingHole_3.2mm_M3" H 7900 5250 50  0001 C CNN
+F 3 "~" H 7900 5250 50  0001 C CNN
+	1    7900 5250
+	1    0    0    -1
+$EndComp
+$Comp
+L Mechanical:MountingHole H2
+U 1 1 61721E3F
+P 7900 5850
+F 0 "H2" H 8000 5896 50  0000 L CNN
+F 1 "MountingHole" H 8000 5805 50  0000 L CNN
+F 2 "MountingHole:MountingHole_3.2mm_M3" H 7900 5850 50  0001 C CNN
+F 3 "~" H 7900 5850 50  0001 C CNN
+	1    7900 5850
+	1    0    0    -1
+$EndComp
+$Comp
+L Mechanical:MountingHole H3
+U 1 1 6172253A
+P 9000 5750
+F 0 "H3" H 9100 5796 50  0000 L CNN
+F 1 "MountingHole" H 9100 5705 50  0000 L CNN
+F 2 "MountingHole:MountingHole_3.2mm_M3" H 9000 5750 50  0001 C CNN
+F 3 "~" H 9000 5750 50  0001 C CNN
+	1    9000 5750
+	1    0    0    -1
+$EndComp
 $EndSCHEMATC
